File: Hardware/Fundbio.sch (KiCad schematic (older format))
At the start: 17 parts, among them M1 Motor, M2 Motor, M3 Motor, Q1 Transistor NPN, Q2 Transistor NPN, Q3 Transistor NPN, U1 Sensor, U2 Sensor, U3 Sensor, U4 HC-05

Commit message: apk
Connections:
- net +9V: now also A1.30 (VIN)
- net at A1.17 (3V3): now also U4.12 (3V3)
Changed lines of the file:
@@
 P 7500 4200
 F 0 "#PWR?" H 7500 4050 50  0001 C CNN
-F 1 "+9V" H 7515 4373 50  0000 C CNN
+F 1 "+3V" H 7515 4373 50  0000 C CNN
 F 2 "" H 7500 4200 50  0001 C CNN
 F 3 "" H 7500 4200 50  0001 C CNN
@@
 L power:+9V #PWR?
 U 1 1 61859BFE
-P 8000 4200
-F 0 "#PWR?" H 8000 4050 50  0001 C CNN
-F 1 "+9V" H 8015 4373 50  0000 C CNN
-F 2 "" H 8000 4200 50  0001 C CNN
-F 3 "" H 8000 4200 50  0001 C CNN
-	1    8000 4200
+P 4150 3600
+F 0 "#PWR?" H 4150 3450 50  0001 C CNN
+F 1 "+9V" H 4165 3773 50  0000 C CNN
+F 2 "" H 4150 3600 50  0001 C CNN
+F 3 "" H 4150 3600 50  0001 C CNN
+	1    4150 3600
 	1    0    0    -1
 $EndComp
@@
 P 8600 4200
 F 0 "#PWR?" H 8600 4050 50  0001 C CNN
-F 1 "+9V" H 8615 4373 50  0000 C CNN
+F 1 "+3V" H 8615 4373 50  0000 C CNN
 F 2 "" H 8600 4200 50  0001 C CNN
 F 3 "" H 8600 4200 50  0001 C CNN
@@
 	1    0    0    -1
 $EndComp
+Wire Wire Line
+	5050 5350 5250 5350
+Wire Wire Line
+	5250 5350 5250 4050
+Wire Wire Line
+	5250 4050 4700 4050
+Wire Wire Line
+	4700 4050 4700 3400
+Wire Wire Line
+	4700 3400 4850 3400
+Wire Wire Line
+	4850 3600 4150 3600
+$Comp
+L power:+9V #PWR?
+U 1 1 6195BAD0
+P 8000 4200
+F 0 "#PWR?" H 8000 4050 50  0001 C CNN
+F 1 "+3V" H 8015 4373 50  0000 C CNN
+F 2 "" H 8000 4200 50  0001 C CNN
+F 3 "" H 8000 4200 50  0001 C CNN
+	1    8000 4200
+	1    0    0    -1
+$EndComp
